Commit message: added parameters, modified parameter values in vesc and lidar driver. Added imu frame. Clean global launch file

File: tf_publisher/launch/ego_racecar.xacro (robot description, xacro)
@@ -12,4 +12,7 @@
   <xacro:property name="laser_radius" value="0.026" />
   <xacro:property name="car_name" value="ego_racecar" />
+  <xacro:property name="imu_x" value="0.15"/>
+  <xacro:property name="imu_y" value="0.0"/>
+  <xacro:property name="imu_z" value="${ground_offset + height}"/>
   <material name="black">
     <color rgba="0.2 0.2 0.2 1."/>
@@ -36,4 +39,17 @@
       <geometry>
         <cylinder radius="${laser_radius}" length="${laser_height}"/>
+      </geometry>
+      <material name="black"/>
+    </visual>
+  </link>
+  <joint name="base_to_imu" type="fixed">
+    <parent link="${car_name}/base_link"/>
+    <child link="${car_name}/imu"/>
+    <origin xyz="${imu_x} ${imu_y} ${imu_z}" rpy="0 0 0"/>
+  </joint>
+  <link name="${car_name}/imu">
+    <visual>
+      <geometry>
+        <box size="0.03 0.03 0.01"/>
       </geometry>
       <material name="black"/>

Commit message: working ekf, slam, amcl

File: tf_publisher/launch/ego_racecar.xacro (robot description, xacro)
@@ -32,8 +32,8 @@
   <joint name="base_to_laser_model" type="fixed">
     <parent link="${car_name}/base_link"/>
-    <child link="${car_name}/laser_model"/>
+    <child link="${car_name}/laser"/>
     <origin xyz="${laser_distance_from_base_link} 0 ${ground_offset+height+(laser_height/2)}"/>
   </joint>
-  <link name="${car_name}/laser_model">
+  <link name="${car_name}/laser">
     <visual>
       <geometry>
